Commit message: Add link to livox_frame

File: src/spot_description_config/spot_macro.xacro (robot description, xacro)
@@ -543,4 +543,5 @@
        <!-- Tassen -->
         <xacro:include filename="$(find spot_description)/urdf/tassen.urdf.xacro" />
+        <xacro:use_tassen tf_prefix="${tf_prefix}" />
         <!-- Optional custom includes. -->
         <xacro:property name="default_empty_urdf" value="$(find spot_description)/urdf/empty.urdf" />

File: src/spot_description_config/tassen.urdf.xacro (robot description, xacro)
@@ -1,46 +1,55 @@
 <?xml version="1.0"?>
 <robot xmlns:xacro="http://www.ros.org/wiki/xacro">
-  <xacro:if value="$(optenv TASSEN 1)">
-    <joint name="tassen_joint" type="fixed">
-      <parent link="front_rail"/>
-      <child link="tassen"/>
-      <origin xyz="-0.035 0 0" rpy="0 0 0"/>
-    </joint>
-    <link name="tassen">
-      <visual>
-        <geometry>
-          <mesh filename="package://spot_description/meshes/tassen/Tassen.obj" scale="0.01 0.01 0.01"/>
-        </geometry>
-      </visual>
-      <collision>
-        <geometry>
-          <mesh filename="package://spot_description/meshes/tassen/TassenProtect.obj" scale="0.01 0.01 0.01"/>
-        </geometry>
-      </collision>
-    </link>
-    <joint name="ZED_mount_joint" type="fixed">
-      <parent link="tassen"/>
-      <child link="ZED_camera"/>
-      <origin xyz="0.06175 0 0.08525" rpy="0 0 0"/>
-    </joint>
-    <link name="ZED_camera">
-      <visual>
-        <geometry>
-          <mesh filename="package://spot_description/meshes/ZED/ZED.obj" scale="0.01 0.01 0.01"/>
-        </geometry>
-      </visual>
-    </link>
-     <joint name="LIVOX_mount_joint" type="fixed">
-      <parent link="tassen"/>
-      <child link="LIVOX_lidar"/>
-      <origin xyz="0 0 0.11925" rpy="0 0 0"/>
-    </joint>
-    <link name="LIVOX_lidar">
-      <visual>
-        <geometry>
-          <mesh filename="package://spot_description/meshes/LIVOX/LIVOX.obj" scale="0.01 0.01 0.01"/>
-        </geometry>
-      </visual>
-    </link>
-  </xacro:if>
+  <!-- Argumenter -->
+  <xacro:macro name="use_tassen" params="tf_prefix">
+    <xacro:if value="$(optenv TASSEN 1)">
+      <joint name="${tf_prefix}tassen_joint" type="fixed">
+        <parent link="${tf_prefix}front_rail"/>
+        <child link="${tf_prefix}tassen"/>
+        <origin xyz="-0.035 0 0" rpy="0 0 0"/>
+      </joint>
+      <link name="${tf_prefix}tassen">
+        <visual>
+          <geometry>
+            <mesh filename="package://spot_description/meshes/tassen/Tassen.obj" scale="0.01 0.01 0.01"/>
+          </geometry>
+        </visual>
+        <collision>
+          <geometry>
+            <mesh filename="package://spot_description/meshes/tassen/TassenProtect.obj" scale="0.01 0.01 0.01"/>
+          </geometry>
+        </collision>
+      </link>
+      <joint name="${tf_prefix}zed_mount_joint" type="fixed">
+        <parent link="${tf_prefix}tassen"/>
+        <child link="${tf_prefix}zed_camera"/>
+        <origin xyz="0.06175 0 0.08525" rpy="0 0 0"/>
+      </joint>
+      <link name="${tf_prefix}zed_camera">
+        <visual>
+          <geometry>
+            <mesh filename="package://spot_description/meshes/ZED/ZED.obj" scale="0.01 0.01 0.01"/>
+          </geometry>
+        </visual>
+      </link>
+      <joint name="${tf_prefix}livox_mount_joint" type="fixed">
+        <parent link="${tf_prefix}tassen"/>
+        <child link="${tf_prefix}livox_lidar"/>
+        <origin xyz="0 0 0.11925" rpy="0 0 0"/>
+      </joint>
+      <link name="${tf_prefix}livox_lidar">
+        <visual>
+          <geometry>
+            <mesh filename="package://spot_description/meshes/LIVOX/LIVOX.obj" scale="0.01 0.01 0.01"/>
+          </geometry>
+        </visual>
+      </link>
+      <joint name="${tf_prefix}lidar_frame" type="fixed">
+        <parent link="${tf_prefix}livox_lidar"/>
+        <child link="livox_frame"/>
+        <origin xyz="0 0 0.47" rpy="0 0 0"/>
+      </joint>
+      <link name="livox_frame"/>
+    </xacro:if>
+  </xacro:macro>
 </robot>
