Commit message: Corected livox_frame transformation distance

File: src/spot_description_config/tassen.urdf.xacro (robot description, xacro)
@@ -48,5 +48,5 @@
         <parent link="${tf_prefix}livox_lidar"/>
         <child link="livox_frame"/>
-        <origin xyz="0 0 0.47" rpy="0 0 0"/>
+        <origin xyz="0 0 0.047" rpy="0 0 0"/>
       </joint>
       <link name="livox_frame"/>

Commit message: Add zed2i

File: src/spot_description_config/tassen.urdf.xacro (robot description, xacro)
@@ -51,4 +51,10 @@
       </joint>
       <link name="livox_frame"/>
+      <joint name="${tf_prefix}zed_camera" type="fixed">
+        <parent link="${tf_prefix}zed_camera"/>
+        <child link="zed_camera_link"/>
+        <origin xyz="0 0 0.047" rpy="0 0 0"/>
+      </joint>
+      <link name="zed_camera_link"/>
     </xacro:if>
   </xacro:macro>

Commit message: Add ca value fore hight

File: src/spot_description_config/tassen.urdf.xacro (robot description, xacro)
@@ -54,5 +54,5 @@
         <parent link="${tf_prefix}zed_camera"/>
         <child link="zed_camera_link"/>
-        <origin xyz="0 0 0.047" rpy="0 0 0"/>
+        <origin xyz="0 0 0.01" rpy="0 0 0"/>
       </joint>
       <link name="zed_camera_link"/>

Commit message: Added the spot pack to the robot description

File: src/spot_description_config/tassen.urdf.xacro (robot description, xacro)
@@ -45,4 +45,21 @@
         </visual>
       </link>
+      <joint name="${tf_prefix}Spotpack" type="fixed">
+        <parent link="${tf_prefix}tassen"/>
+        <child link="${tf_prefix}SpotPack"/>
+        <origin xyz="-0.2425 0 0" rpy="0 0 0"/>
+      </joint>
+      <link name="${tf_prefix}SpotPack">
+        <visual>
+          <geometry>
+            <mesh filename="package://spot_description/meshes/SpotPack/SpotPack.obj" scale="0.01 0.01 0.01"/>
+          </geometry>
+        </visual>
+        <collision>
+          <geometry>
+            <mesh filename="package://spot_description/meshes/SpotPack/SpotPackCollision.obj" scale="0.01 0.01 0.01"/>
+          </geometry>
+        </collision>
+      </link>
       <joint name="${tf_prefix}lidar_frame" type="fixed">
         <parent link="${tf_prefix}livox_lidar"/>
